File: Schaltung/Schaltplan.brd (EAGLE design)
At the start: 100 x 60 mm, 52 parts, among them IC1 ATMEGA1284P, IC3 LP 2950(turn_around), Q1 8MHz, Q2 32.786kHz, Q3 BS170, Q4 BS170, Q5 BC547B, Q6 BC557B

Commit message: Schaltplan/Board beim Hersteller hochgeladen
Parts:
- removed DRILEGEND: (no value), drilegend:DRILEGEND
- added R14, R15: 100k, rcl:0207/10
- moved R13 63.5 mm to (19.1, 41.9), turned to 270 degrees
- moved HMC5883L 2.54 mm to (20.3, 12.7)
- moved BOARD 1.27 mm to (10.2, 12.7), turned to 90 degrees
- moved IR 1.27 mm to (19.1, 22.9)
- moved R10 1.27 mm to (22.9, 20.3)
- moved S1 1.27 mm to (45.7, 48.3)
Connections:
- net GND: now also R13.1, R14.1, R15.1
- net N$11: now also R13.2
- net N$12: now also R14.2
- net N$13: now also R15.2
Routing:
- net GND: track 298.7 -> 316.1 mm
- net CARD-DETECT: track 64.8 -> 81.0 mm
- net +3V3: track 202.1 -> 217.8 mm
- net FIX: track 27.3 -> 41.5 mm
- net EN: track 28.2 -> 41.7 mm
- net N$11: track 27.6 -> 38.6 mm
- net N$12: track 24.1 -> 28.9 mm
- net SCK: track 77.1 -> 72.5 mm
- net SCL: track 28.0 -> 31.5 mm
- net SDA: track 29.4 -> 32.7 mm
- net N$13: track 24.9 -> 22.0 mm
- net MOSI: track 69.9 -> 71.4 mm
- net N$19: track 5.63 -> 4.44 mm
- net MISO: track 65.2 -> 64.1 mm
- net N$6: track 11.7 -> 12.7 mm
